File: PFIP PCB/PFIP PCB/PFIP PCB.kicad_sch (KiCad schematic)
At the start: 15 parts, among them M1 Motor_Servo, P1 STEP DOWN, P2 MAIN, P3 LOAD, P4 220V-24V_Power_Supply, P5 PZEM-004T, P6 Step_Down_Module, SW1 SW_Push, SW2 PWR SW, T1 CST1_Split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

Commit message: Icon and App name Change
Parts:
- removed M1: Motor_Servo, Connector_JST:JST_EH_B3B-EH-A_1x03_P2.50mm_Vertical, symbol Motor:Motor_Servo
- added P7: BULB, symbol Connector:Conn_WallPlug
- added R2: RELAY, symbol Custom Library:1_Channel_Relay_Module
- P3: value LOAD -> FAN
Connections:
- net +5V: now also R2.1 (VCC)
- net GND: now also R2.2 (GND)
- net at P2.2 (AC_N), P3.2 (AC_N), P4. (24VDC_-)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: now also P7.2 (AC_N)
- net AC_P1: now reaches P2.1 (AC_P), P4. (24VDC_-), P5.8 (AC_L), U2.4
- net AC_P1: now also R2. (NO)
- net SERVO renamed REL_IN
- net REL_IN: now also R2.3 (IN1)
- new net AC_P2: P7.1 (AC_P), R2. (NO)
- no-connect marks 0 -> 1
Other:
- moved on the sheet: U2
